File: SynthLabBadge/SynthLabBadge.kicad_pcb (KiCad board)
At the start: 2 copper layers, 128.5 x 40.3 mm, 72 parts, among them J2 Probe In, J3 Mix_In, J4 Out, J5 Eurorack_Power_10pin_Unshroud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, J6 Mix In, J7 Probe, J8 Conn_Out, J9 Vol Pot, U1 LM358, U2 CD40106BPWR

Commit message: final check before production
Parts:
- removed the REF** at (52.0, 127.8)
- removed the REF** at (174.5, 99.8)
- added ?: , , F.Cu at (52.0, 125.4)
- added REF**: logo_fablabnk, Library:logo_fablabnk, F.Cu at (65.6, 124.6)
- added REF**: logo_42berlin, Library:logo_42berlin, B.Cu at (70.8, 126.4)
Routing:
- net Net-(U2D-I): track 103.3 -> 106.6 mm
- net Net-(U2E-I): track 82.4 -> 83.8 mm, vias 0 -> 2
- net Net-(U2F-I): track 81.5 -> 82.5 mm
- net Net-(J7-Pin_1): track 91.0 -> 91.8 mm, vias 4 -> 6
- net Net-(U2A-I): track 100.2 -> 100.7 mm
- net Net-(U2B-O): track 91.6 -> 91.8 mm, vias 4 -> 6
Other:
- outline, holes or cut-outs redrawn
- board text added: "BY 42 BERLIN SYNTHLAB"
- board text added: "DESIGNED AT"
- board text added: "INSPIRED BY DYLAN B. BEAM CATCHER"
- board text added: "JLCJLCJLCJLC"
- board text added: "SUPPORTED BY"
- board text added: "loess-labs.net/ inst/beam/"
- board text added: "workish.berlin/ synthlab"
