File: SynthLabBadge.kicad_pcb (KiCad board)
At the start: 2 copper layers, 128.5 x 40.3 mm, 73 parts, among them J2 Probe In, J3 Mix_In, J4 Out, J5 Eurorack_Power_10pin_Unshroud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, J6 Mix In, J7 Probe, J8 Conn_Out, J9 Vol Pot, U1 LM358, U2 CD40106BPWR

Commit message: commiting before trying to move components from bottom of board
Parts:
- added ?: , , F.Cu at (174.5, 99.9)
- added BatteryMount: 9VBatteryClop, Library:9VBatteryClop, B.Cu at (120.7, 114.9)
- added R20: 100K, Resistor_THT:R_Axial_DIN0207_L6.3mm_D2.5mm_P10.16mm_Horizontal, B.Cu at (121.8, 129.4)
- BT1: value 9V Bat -> 9V Battery
- J3: value Mix_In -> Mix In
- J7: value Probe -> Probe In
- J8: value Conn_Out -> Out
- JP1: value Jump4Stereo -> Jmp4Stereo
- R14, R15, R16, R17, R18, R19: value 100k -> 1k
- R4: value 500k1M -> 10k
- moved C11 34.2 mm to (97.1, 100.0)
- moved BT1 33.7 mm to (95.2, 104.6), turned to 171.5 degrees
- moved R4 30.5 mm to (150.2, 129.4), turned to 180 degrees
- moved J8 29.7 mm to (171.5, 124.2), turned to 171.5 degrees
- moved R13 24.4 mm to (101.1, 114.5), turned to 180 degrees
- moved J9 21.8 mm to (164.7, 102.5), turned to 81.5 degrees
- moved C9 20.1 mm to (132.3, 110.3), turned to 0 degrees
- moved R14 14.8 mm to (53.4, 110.3), turned to 0 degrees
- moved J7 13.9 mm to (62.7, 96.7), turned to 171.5 degrees
- moved R2 10.2 mm to (89.6, 100.1), turned to -98.5 degrees
- moved R1 10.2 mm to (76.2, 100.2), turned to -98.5 degrees
- moved R8 10.2 mm to (103.8, 100.2), turned to -98.5 degrees
- moved R15 10.1 mm to (99.2, 110.2), turned to 81.5 degrees
- moved mouse-bite-1mm-slot 9.28 mm to (127.6, 96.2)
- moved R3 8.87 mm to (168.5, 121.3), turned to -98.5 degrees
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Connections:
- BT1 pad 1: VCC -> Net-(BT1-+)
- C11 pad 1: VCC -> Net-(BT1-+)
- D8 pad 2: Net-(D8-A) -> Net-(BT1-+)
- J5 pad 1: Net-(D8-A) -> Net-(BT1-+)
- J5 pad 2: Net-(D8-A) -> Net-(BT1-+)
- R1 pad 1: Net-(R1-Pad1) -> Net-(U2A-I)
- R1 pad 2: Net-(U2A-O) -> Net-(R1-Pad2)
- R12 pad 1: Net-(R12-Pad1) -> Net-(U2E-I)
- R12 pad 2: Net-(U2E-O) -> Net-(R12-Pad2)
- R13 pad 1: Net-(R13-Pad1) -> Net-(U2F-I)
- R13 pad 2: Net-(U2F-O) -> Net-(R13-Pad2)
- R2 pad 1: Net-(R2-Pad1) -> Net-(U2B-I)
- R2 pad 2: Net-(U2B-O) -> Net-(R2-Pad2)
- R8 pad 1: Net-(R8-Pad1) -> Net-(U2C-I)
- R8 pad 2: Net-(U2C-O) -> Net-(R8-Pad2)
- R9 pad 1: Net-(R9-Pad1) -> Net-(U2D-I)
- R9 pad 2: Net-(U2D-O) -> Net-(R9-Pad2)
- RV1 pad 1: Net-(U2A-I) -> unconnected-(RV1-Pad1)
- RV1 pad 2: Net-(U2A-I) -> Net-(R1-Pad2)
- RV1 pad 3: Net-(R1-Pad1) -> Net-(U2A-O)
- RV2 pad 1: Net-(U2B-I) -> unconnected-(RV2-Pad1)
- RV2 pad 2: Net-(U2B-I) -> Net-(R2-Pad2)
- RV2 pad 3: Net-(R2-Pad1) -> Net-(U2B-O)
- RV4 pad 1: Net-(U2C-I) -> unconnected-(RV4-Pad1)
- RV4 pad 2: Net-(U2C-I) -> Net-(R8-Pad2)
- RV4 pad 3: Net-(R8-Pad1) -> Net-(U2C-O)
- RV5 pad 1: Net-(U2D-I) -> unconnected-(RV5-Pad1)
- RV5 pad 2: Net-(U2D-I) -> Net-(R9-Pad2)
- RV5 pad 3: Net-(R9-Pad1) -> Net-(U2D-O)
- RV6 pad 1: Net-(U2E-I) -> unconnected-(RV6-Pad1)
- RV6 pad 2: Net-(U2E-I) -> Net-(R12-Pad2)
- RV6 pad 3: Net-(R12-Pad1) -> Net-(U2E-O)
- RV7 pad 1: Net-(U2F-I) -> unconnected-(RV7-Pad1)
- RV7 pad 2: Net-(U2F-I) -> Net-(R13-Pad2)
- RV7 pad 3: Net-(R13-Pad1) -> Net-(U2F-O)
Routing:
- net Net-(R12-Pad2): track 0.00 -> 53.9 mm, vias 0 -> 4
- net Net-(R9-Pad2): track 0.00 -> 53.0 mm, vias 0 -> 4
- net Net-(U2E-O): track 20.7 -> 73.4 mm, vias 2 -> 0
- net Net-(U2D-I): track 106.6 -> 59.4 mm, vias 10 -> 2
- net Net-(U2D-O): track 34.8 -> 78.9 mm, vias 2 -> 8
- net Net-(R12-Pad1): track 42.5 -> 0.00 mm, vias 2 -> 0
- net Net-(U2F-O): track 27.2 -> 67.4 mm
- net Net-(R9-Pad1): track 36.7 -> 0.00 mm
- net Net-(U2A-O): track 93.4 -> 128.5 mm, vias 4 -> 7
- net Net-(BT1-+): track 0.00 -> 34.0 mm
- net Net-(U2F-I): track 82.5 -> 50.3 mm
- net Net-(R4-Pad2): track 34.8 -> 66.8 mm, vias 0 -> 1
- net Net-(U2E-I): track 83.8 -> 53.3 mm, vias 2 -> 3
- net Net-(U2C-O): track 54.3 -> 84.2 mm
- net Net-(J8-Pin_1): track 10.3 -> 34.9 mm, vias 0 -> 2
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Other:
- outline, holes or cut-outs redrawn
- board text added: "BATTERY POWER AT SAME TIME!"
- board text added: "Mix In▲"
- board text added: "NEVER CONNECT EURORACK &"
- board text added: "Out▲"
- board text added: "Probe In►"
- board text added: "V1.1"
- board text added: "Vol▼"
- board text removed: "V1.0"

Commit message: V1.1 ready for production
Parts:
- removed JP1: Jmp4Stereo, Jumper:SolderJumper-2_P1.3mm_Open_RoundedPad1.0x1.5mm
- R1, R10, R11, R12, R13, R14, R15, R16, R17, R18, R19, R2, R20, R3, R4, R5, R6, R7, R8, R9: footprint Resistor_THT:R_Axial_DIN0207_L6.3mm_D2.5mm_P10.16mm_Horizontal -> Resistor_THT:R_Axial_DIN0207_L6.3mm_D2.5mm_P2.54mm_Vertical
- moved R14 54.8 mm to (107.4, 101.4)
- moved C2 48.0 mm to (117.8, 129.3), turned to 0 degrees
- moved R17 44.2 mm to (132.8, 110.3), turned to 0 degrees
- moved R15 40.2 mm to (139.3, 107.9), turned to -98.5 degrees
- moved R9 37.2 mm to (75.2, 106.2), turned to -98.5 degrees
- moved R12 36.1 mm to (89.3, 106.2), turned to -98.5 degrees
- moved R6 33.2 mm to (140.9, 129.3), turned to 180 degrees
- moved R3 32.2 mm to (136.3, 121.5), turned to 81.5 degrees
- moved D8 29.1 mm to (85.4, 114.5), turned to 0 degrees
- moved R16 29.0 mm to (130.7, 129.3), turned to 180 degrees
- moved C7 29.0 mm to (126.6, 100.9), turned to -98.5 degrees
- moved C8 28.6 mm to (116.8, 100.9)
- moved J8 26.9 mm to (145.1, 129.3), turned to -90 degrees
- moved C3 24.9 mm to (127.0, 119.0), turned to -98.5 degrees
- moved C4 24.8 mm to (129.8, 100.9), turned to -98.5 degrees
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Connections:
- J8 pad T: Net-(J8-Pin_2) -> Net-(J8-Pin_1)
- R11 pad 2: Net-(J8-Pin_2) -> Net-(J8-Pin_1)
Routing:
- net VCC: track 88.3 -> 195.1 mm, vias 0 -> 1
- net Net-(J8-Pin_2): track 58.4 -> 0.00 mm, vias 2 -> 0
- net Net-(D2-A): track 47.4 -> 5.06 mm
- net Net-(R11-Pad1): track 60.7 -> 20.0 mm, vias 6 -> 0
- net Net-(U2A-O): track 128.5 -> 89.4 mm, vias 7 -> 11
- net Net-(R4-Pad2): track 66.8 -> 30.6 mm, vias 1 -> 0
- net Net-(U1A-+): track 7.13 -> 40.9 mm, vias 0 -> 4
- net Net-(D4-A): track 36.9 -> 5.79 mm
- net Net-(R12-Pad2): track 53.9 -> 23.0 mm, vias 4 -> 0
- net Net-(D3-A): track 47.1 -> 17.1 mm, vias 1 -> 0
- net Net-(U2D-I): track 59.4 -> 88.6 mm, vias 2 -> 12
- net Net-(J8-Pin_1): track 34.9 -> 7.09 mm, vias 2 -> 0
- net Net-(R9-Pad2): track 53.0 -> 25.7 mm, vias 4 -> 0
- net Net-(U2C-O): track 84.2 -> 57.2 mm, vias 4 -> 7
- net Net-(D7-A): track 26.7 -> 6.16 mm
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Other:
- board text added: "Mix In ▼"
- board text added: "Out ▲"
- board text added: "Probe In ►"
- board text added: "Vol ▲"
- board text removed: "Mix In▲"
- board text removed: "Out▲"
- board text removed: "Probe In►"
- board text removed: "Vol▼"

Commit message: V1.1 ready for production
Parts:
- R20: value 100K -> 100k
- R6: value 1k -> 1.5k

Commit message: All 3D models added and positioned - ready to create build guide
Parts:
- C1, C10, C2, C3, C4, C5, C6, C7, C8, C9: footprint Capacitor_THT:C_Axial_L3.8mm_D2.6mm_P7.50mm_Horizontal -> Library:C_Axial_L3.8mm_D2.6mm_P7.50mm_Horizontal_Disc3DModel
- D2, D3, D4, D5, D6, D7: footprint LED_THT:LED_D5.0mm -> Library:LED_D5.0mm_Lowered
- RV1, RV2, RV4, RV5, RV6, RV7: footprint Potentiometer_THT:Potentiometer_Runtron_RM-065_Vertical -> Library:Potentiometer_Runtron_RM-065_Vertical_With3DModel
