File: SynthLabBadge.kicad_sch (KiCad schematic)
At the start: 58 parts, among them J1 Probe Out, J2 Probe In, J3 Mix_In, J4 Out, J5 Eurorack_Power_10pin_Unshroud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, J6 Conn_Mix_In, J7 Conn_Probe, J8 Conn_Out, J9 Conn_Vol_Pot, U1 LM358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

Commit message: commiting before trying to move components from bottom of board
Parts:
- added R20: 100K, Resistor_THT:R_Axial_DIN0207_L6.3mm_D2.5mm_P10.16mm_Horizontal, symbol Device:R
- D8: value 1N5817 -> 5817
- J3: value Mix_In -> Mix In
- J4: symbol Connector_Audio:AudioJack2_SwitchT -> Connector_Audio:AudioJack3
- J6: value Conn_Mix_In -> Mix In
- J7: value Conn_Probe -> Probe In
- J8: value Conn_Out -> Out
- J9: value Conn_Vol_Pot -> Vol Pot
- JP1: value Jumper_2_Open -> Jmp4Stereo
- R14, R15, R16, R17, R18, R19: value 100k -> 1k
- R4: value 500k-1M -> 10k
Connections:
- net VCC: now also R20.2; no longer BT1.1 (+), C11.1
- net at C6.1, U2.5 (I): now also R8.1; no longer RV4.1, RV4.2
- net at RV4.3: now also R15.1, U2.6 (O); no longer R8.1
- net at C4.1, U2.1 (I): now also R1.1; no longer RV1.1, RV1.2
- net at R14.1, U2.2 (O): now also RV1.3; no longer R1.2
- net at R19.1, U2.12 (O): now also RV7.3; no longer R13.2
- net at C9.1, U2.13 (I): now also R13.1; no longer RV7.1, RV7.2
- net at C8.1, U2.11 (I): now also R12.1; no longer RV6.1, RV6.2
- net at RV6.3: now also R16.1, U2.10 (O); no longer R12.1
- net at C7.1, U2.9 (I): now also R9.1; no longer RV5.1, RV5.2
- net at RV5.3: now also R18.1, U2.8 (O); no longer R9.1
- net at R2.1: now also C5.1, U2.3 (I); no longer RV2.3
- net at R17.1, U2.4 (O): now also RV2.3; no longer R2.2
- net at C1.1, D1.2 (A), J1.T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: now also R20.1
- net at D8.2 (A), J5.1 (+12V), J5.2 (+12V): now also BT1.1 (+), C11.1
- new net: R8.2, RV4.2
- new net: R12.2, RV6.2
- new net: R9.2, RV5.2
- new net: R13.2, RV7.2
- new net: R2.2, RV2.2
- new net: J4.R, J8.R (Pin_1), JP1.2 (B)
- new net: R1.2, RV1.2
- now unconnected: RV2.1
- no-connect marks 4 -> 10
Other:
- note added: "Bridge this with solder if using a stereo 3.5mm output jack (headphones) or leave open if using a switched mono output jack (footprint is the same - TN turns to R)"
- note added: "Can be +9V or +12V Original Beam Catcher is +5V"
- note added: "needed?"
- note removed: "Bridge if not wanted"
- note removed: "Bridge this with solder if using a stereo 3.5mm output jack (headphones) or leave open if using a switched mono output jack (footprint is the same)"
- note removed: "Can be +9V or +12V"
- moved on the sheet: D8, R1, R12, R13, R2, R3, R8, R9

Commit message: V1.1 ready for production
Parts:
- removed JP1: Jmp4Stereo, Jumper:SolderJumper-2_P1.3mm_Open_RoundedPad1.0x1.5mm, symbol Jumper:Jumper_2_Open
- R1, R10, R11, R12, R13, R14, R15, R16, R17, R18, R19, R2, R20, R3, R4, R5, R6, R7, R8, R9: footprint Resistor_THT:R_Axial_DIN0207_L6.3mm_D2.5mm_P10.16mm_Horizontal -> Resistor_THT:R_Axial_DIN0207_L6.3mm_D2.5mm_P2.54mm_Vertical
Connections:
- net at J4.R, J8.R (Pin_1): now also J4.T, J8.T (Pin_2), R11.2
Other:
- note added: "Can you stereo 3.5mm output jack or switched thonkiconn mono jack here (R turns to TN)"
- note removed: "- will stereo jack idea work? Does R replace TN or T? - 47uF or 22uF - check which way around pot should be - add clip slot! - 9V battery dimensions = 48.5mm x 26.5mm x 17.5mm - battery placement off board for now. In V2 SMT components might be on front and we find space for it on back. - thonkiconn mounting: jack socket is screwed to pcb and is point-to-point wired to mounting holes on PCB - whe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"
- note removed: "Bridge this with solder if using a stereo 3.5mm output jack (headphones) or leave open if using a switched mono output jack (footprint is the same - TN turns to R)"
- note removed: "Practical notes - changing from 9V to 12V affects pitch, but it still tunable within a nice range - sides of thonkiconn photodiode probe need to be held otherwise output is V quiet - pot is wired wrong way around on breadboard - check this in schematic - line input can be given as a test but overloads, so reduce volume - above dual op amp approach works but first op amp could amplify the probe mo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"
- note removed: "needed?"
- note removed: "summing configuration: equal value resistors on both inputs going to minus and in the loop"
Changed lines of the file:
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@@
 	(generator_version "9.0")
 	(paper "A4")
-	(text "needed?"
-		(exclude_from_sim no)
-		(at 276.352 33.02 0)
-		(effects
-			(font
-				(size 1.27 1.27)
-			)
-		)
-	)
 	(text "Output of another beam catcher badge\ncan be fed in here, to mix two sets of\noscillators.original beam catcher\n- In original one goes to left, one goes to right output"
 		(exclude_from_sim no)
-		(at 133.35 72.39 0)
+		(at 167.386 90.424 0)
 		(effects
 			(font
 				(size 1.27 1.27)
 			)
+			(justify left)
 		)
 	)
@@
 		)
 	)
-	(text "Bridge this with solder\nif using a stereo 3.5mm\noutput jack (headphones)\nor leave open if using a\nswitched mono output jack\n(footprint is the same - TN turns to R)"
+	(text "Can you stereo 3.5mm\noutput jack or\nswitched thonkiconn\nmono jack here\n(R turns to TN)"
 		(exclude_from_sim no)
-		(at 239.268 59.436 0)
+		(at 270.256 64.008 0)
 		(effects
 			(font
@@
 		)
 	)
-	(text "Practical notes\n- changing from 9V to 12V affects pitch, but it still tunable within a nice range\n- sides of thonkiconn photodiode probe need to be held otherwise output is V quiet\n- pot is wired wrong way around on breadboard - check this in schematic\n- line input can be given as a test but overloads, so reduce volume\n- above dual op amp approach works but first op amp could amplify the probe more\n- trimpot is not very tunable (would changing 1k resistor here make a difference)"
-		(exclude_from_sim no)
-		(at 152.146 146.558 0)
-		(effects
-			(font
-				(size 1.27 1.27)
-			)
-			(justify left)
-		)
-	)
 	(text "Can be +9V or +12V\nOriginal Beam Catcher is +5V"
 		(exclude_from_sim no)
@@
 		)
 	)
-	(text "- will stereo jack idea work? Does R replace TN or T?\n- 47uF or 22uF\n- check which way around pot should be\n- add clip slot!\n- 9V battery dimensions = 48.5mm x 26.5mm x 17.5mm\n- battery placement off board for now. In V2 SMT components might be on front and we find space for it on back.\n- thonkiconn mounting: jack socket is screwed to pcb and is point-to-point wired to mounting holes on PCB\n- where could battery be mounted? is clip possible?\n- 100k resistor has been added between op amp output and LED\n	- not shown here: https://github.com/uvknhn/Beam-Catcher/blob/main/v1/schematic.png !\n- will mixer chaining approach work?\n	- how it works:\n	- a photodiode is on the end of probe cable which plugs into a thonkiconn and goes to plus input of first LM358\n	- output of LM358 goes into minus input of second LM358\n	- Out of other badge goes to thonkiconn Mix In of this badge, which in turn goes to minus input of second LM358\n	- mixed output goes to Out thonkiconn\n	- either a mono or stereo thonkiconn can be used at Out. When stereo output jumper needs to be bridged\n- will +9V/+12V approach work? Yes, both chips can operate with 12V\n- choose PCB colour: red,yellow,blue\n- route it\n- silkscreen component values\n- silkscreen connectors (i.e. T R S)\n- add eurorack screw slots\n- V2: go SMT! Would be more electrically sound (no solder connections on front side of badge)"
-		(exclude_from_sim no)
-		(at 150.876 113.792 0)
-		(effects
-			(font
-				(size 1.27 1.27)
-			)
-			(justify left)
-		)
-	)
-	(text "summing configuration: equal value resistors on both inputs going to minus and in the loop"
-		(exclude_from_sim no)
-		(at 193.548 88.138 0)
-		(effects
-			(font
-				(size 1.27 1.27)
-			)
-		)
-	)
 	(junction
 		(at 17.78 86.36)
@@
 	)
 	(junction
-		(at 233.68 73.66)
-		(diameter 0)
-		(color 0 0 0 0)
-	)
-	(junction
 		(at 149.86 34.29)
 		(diameter 0)
@@
 	)
 	(junction
+		(at 233.68 73.66)
+		(diameter 0)
+		(color 0 0 0 0)
+	)
+	(junction
 		(at 171.45 44.45)
 		(diameter 0)
@@
 	(wire
 		(pts
+			(xy 233.68 73.66) (xy 243.84 73.66)
+		)
+		(stroke
+			(width 0)
+			(type default)
+		)
+	)
+	(wire
+		(pts
 			(xy 66.04 130.81) (xy 66.04 132.08)
 		)
@@
 			)
 		)
-		(property "Footprint" "Resistor_THT:R_Axial_DIN0207_L6.3mm_D2.5mm_P10.16mm_Horizontal"
+		(property "Footprint" "Resistor_THT:R_Axial_DIN0207_L6.3mm_D2.5mm_P2.54mm_Vertical"
 			(at 199.39 72.898 90)
 			(effects
@@
 			)
 		)
-		(property "Footprint" "Resistor_THT:R_Axial_DIN0207_L6.3mm_D2.5mm_P10.16mm_Horizontal"
+		(property "Footprint" "Resistor_THT:R_Axial_DIN0207_L6.3mm_D2.5mm_P2.54mm_Vertical"
 			(at 16.002 74.93 90)
 			(effects
@@
 			)
 		)
-		(property "Footprint" "Resistor_THT:R_Axial_DIN0207_L6.3mm_D2.5mm_P10.16mm_Horizontal"
+		(property "Footprint" "Resistor_THT:R_Axial_DIN0207_L6.3mm_D2.5mm_P2.54mm_Vertical"
 			(at 46.99 43.688 90)
 			(effects
@@
 			)
 		)
-		(property "Footprint" "Resistor_THT:R_Axial_DIN0207_L6.3mm_D2.5mm_P10.16mm_Horizontal"
+		(property "Footprint" "Resistor_THT:R_Axial_DIN0207_L6.3mm_D2.5mm_P2.54mm_Vertical"
 			(at 173.228 24.13 90)
 			(effects
@@
 			)
 		)
-		(property "Footprint" "Resistor_THT:R_Axial_DIN0207_L6.3mm_D2.5mm_P10.16mm_Horizontal"
+		(property "Footprint" "Resistor_THT:R_Axial_DIN0207_L6.3mm_D2.5mm_P2.54mm_Vertical"
 			(at 64.262 31.75 90)
 			(effects
@@
 			)
 		)
-		(property "Footprint" "Resistor_THT:R_Axial_DIN0207_L6.3mm_D2.5mm_P10.16mm_Horizontal"
+		(property "Footprint" "Resistor_THT:R_Axial_DIN0207_L6.3mm_D2.5mm_P2.54mm_Vertical"
 			(at 16.002 120.65 90)
 			(effects
@@
 			)
 		)
-		(property "Footprint" "Resistor_THT:R_Axial_DIN0207_L6.3mm_D2.5mm_P10.16mm_Horizontal"
+		(property "Footprint" "Resistor_THT:R_Axial_DIN0207_L6.3mm_D2.5mm_P2.54mm_Vertical"
 			(at 199.39 38.608 90)
 			(effects
@@
 			)
 		)
-		(property "Footprint" "Resistor_THT:R_Axial_DIN0207_L6.3mm_D2.5mm_P10.16mm_Horizontal"
+		(property "Footprint" "Resistor_THT:R_Axial_DIN0207_L6.3mm_D2.5mm_P2.54mm_Vertical"
 			(at 16.002 31.75 90)
 			(effects
@@
 			)
 		)
-		(property "Footprint" "Resistor_THT:R_Axial_DIN0207_L6.3mm_D2.5mm_P10.16mm_Horizontal"
+		(property "Footprint" "Resistor_THT:R_Axial_DIN0207_L6.3mm_D2.5mm_P2.54mm_Vertical"
 			(at 210.82 66.548 90)
 			(effects
@@
 			)
 		)
-		(property "Footprint" "Resistor_THT:R_Axial_DIN0207_L6.3mm_D2.5mm_P10.16mm_Horizontal"
+		(property "Footprint" "Resistor_THT:R_Axial_DIN0207_L6.3mm_D2.5mm_P2.54mm_Vertical"
 			(at 46.99 132.588 90)
 			(effects
@@
 			)
 		)
-		(property "Footprint" "Resistor_THT:R_Axial_DIN0207_L6.3mm_D2.5mm_P10.16mm_Horizontal"
+		(property "Footprint" "Resistor_THT:R_Axial_DIN0207_L6.3mm_D2.5mm_P2.54mm_Vertical"
 			(at 64.262 74.93 90)
 			(effects
@@
 			)
 		)
-		(property "Footprint" "Resistor_THT:R_Axial_DIN0207_L6.3mm_D2.5mm_P10.16mm_Horizontal"
+		(property "Footprint" "Resistor_THT:R_Axial_DIN0207_L6.3mm_D2.5mm_P2.54mm_Vertical"
 			(at 95.25 88.138 90)
 			(effects
@@
 			)
 		)
-		(property "Footprint" "Resistor_THT:R_Axial_DIN0207_L6.3mm_D2.5mm_P10.16mm_Horizontal"
+		(property "Footprint" "Resistor_THT:R_Axial_DIN0207_L6.3mm_D2.5mm_P2.54mm_Vertical"
 			(at 95.25 43.688 90)
 			(effects
@@
 			)
 		)
-		(property "Footprint" "Resistor_THT:R_Axial_DIN0207_L6.3mm_D2.5mm_P10.16mm_Horizontal"
+		(property "Footprint" "Resistor_THT:R_Axial_DIN0207_L6.3mm_D2.5mm_P2.54mm_Vertical"
 			(at 224.79 37.592 90)
 			(effects
@@
 			)
 		)
-		(property "Footprint" "Resistor_THT:R_Axial_DIN0207_L6.3mm_D2.5mm_P10.16mm_Horizontal"
+		(property "Footprint" "Resistor_THT:R_Axial_DIN0207_L6.3mm_D2.5mm_P2.54mm_Vertical"
 			(at 224.79 71.882 90)
 			(effects
@@
 			)
 		)
-		(property "Footprint" "Resistor_THT:R_Axial_DIN0207_L6.3mm_D2.5mm_P10.16mm_Horizontal"
+		(property "Footprint" "Resistor_THT:R_Axial_DIN0207_L6.3mm_D2.5mm_P2.54mm_Vertical"
 			(at 46.99 88.138 90)
 			(effects
@@
 	)
 	(symbol
-		(lib_id "Jumper:Jumper_2_Open")
-		(at 238.76 73.66 0)
-		(unit 1)
-		(exclude_from_sim no)
-		(in_bom yes)
-		(on_board yes)
-		(dnp no)
-		(property "Reference" "JP1"
-			(at 238.76 67.31 0)
-			(effects
-				(font
-					(size 1.27 1.27)
-				)
-			)
-		)
-		(property "Value" "Jmp4Stereo"
-			(at 238.76 69.85 0)
-			(effects
-				(font
-					(size 1.27 1.27)
-				)
-			)
-		)
-		(property "Footprint" "Jumper:SolderJumper-2_P1.3mm_Open_RoundedPad1.0x1.5mm"
-			(at 238.76 73.66 0)
-			(effects
-				(font
-					(size 1.27 1.27)
-				)
-				(hide yes)
-			)
-		)
-		(property "Datasheet" "~"
-			(at 238.76 73.66 0)
-			(effects
-				(font
-					(size 1.27 1.27)
-				)
-				(hide yes)
-			)
-		)
-		(property "Description" "Jumper, 2-pole, open"
-			(at 238.76 73.66 0)
-			(effects
-				(font
-					(size 1.27 1.27)
-				)
-				(hide yes)
-			)
-		)
-		(pin "2"
-		)
-		(pin "1"
-		)
-		(instances
-			(project ""
-				(path "/3cb18f4a-e616-4f52-9c11-d7b5d96e6e33"
-					(reference "JP1")
-					(unit 1)
-				)
-			)
-		)
-	)
-	(symbol
 		(lib_id "Device:C")
 		(at 66.04 91.44 0)
@@
 			)
 		)
-		(property "Footprint" "Resistor_THT:R_Axial_DIN0207_L6.3mm_D2.5mm_P10.16mm_Horizontal"
+		(property "Footprint" "Resistor_THT:R_Axial_DIN0207_L6.3mm_D2.5mm_P2.54mm_Vertical"
 			(at 95.25 132.588 90)
 			(effects
@@
 			)
 		)
-		(property "Footprint" "Resistor_THT:R_Axial_DIN0207_L6.3mm_D2.5mm_P10.16mm_Horizontal"
+		(property "Footprint" "Resistor_THT:R_Axial_DIN0207_L6.3mm_D2.5mm_P2.54mm_Vertical"
 			(at 64.262 120.65 90)
 			(effects
@@
 			)
 		)
-		(property "Footprint" "Resistor_THT:R_Axial_DIN0207_L6.3mm_D2.5mm_P10.16mm_Horizontal"
+		(property "Footprint" "Resistor_THT:R_Axial_DIN0207_L6.3mm_D2.5mm_P2.54mm_Vertical"
 			(at 210.82 32.258 90)
 			(effects
@@
 			)
 		)
-		(property "Footprint" "Resistor_THT:R_Axial_DIN0207_L6.3mm_D2.5mm_P10.16mm_Horizontal"
+		(property "Footprint" "Resistor_THT:R_Axial_DIN0207_L6.3mm_D2.5mm_P2.54mm_Vertical"
 			(at 191.262 46.99 90)
 			(effects

Commit message: V1.1 ready for production
Parts:
- R20: value 100K -> 100k
- R6: value 1k -> 1.5k
Changed lines of the file:
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@@
 			)
 		)
-		(property "Value" "100K"
+		(property "Value" "100k"
 			(at 173.99 25.3999 0)
 			(effects
@@
 			)
 		)
-		(property "Value" "1k"
+		(property "Value" "1.5k"
 			(at 224.79 43.18 90)
 			(effects

Commit message: All 3D models added and positioned - ready to create build guide
Parts:
- C1, C10, C2, C3, C4, C5, C6, C7, C8, C9: footprint Capacitor_THT:C_Axial_L3.8mm_D2.6mm_P7.50mm_Horizontal -> Library:C_Axial_L3.8mm_D2.6mm_P7.50mm_Horizontal_Disc3DModel
- D2, D3, D4, D5, D6, D7: footprint LED_THT:LED_D5.0mm -> Library:LED_D5.0mm_Lowered
- RV1, RV2, RV4, RV5, RV6, RV7: footprint Potentiometer_THT:Potentiometer_Runtron_RM-065_Vertical -> Library:Potentiometer_Runtron_RM-065_Vertical_With3DModel
Changed lines of the file:
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@@
 			)
 		)
-		(property "Footprint" "Capacitor_THT:C_Axial_L3.8mm_D2.6mm_P7.50mm_Horizontal"
+		(property "Footprint" "Library:C_Axial_L3.8mm_D2.6mm_P7.50mm_Horizontal_Disc3DModel"
 			(at 135.5852 176.53 0)
 			(effects
@@
 			)
 		)
-		(property "Footprint" "Potentiometer_THT:Potentiometer_Runtron_RM-065_Vertical"
+		(property "Footprint" "Library:Potentiometer_Runtron_RM-065_Vertical_With3DModel"
 			(at 25.4 66.04 0)
 			(effects
@@
 			)
 		)
-		(property "Footprint" "Capacitor_THT:C_Axial_L3.8mm_D2.6mm_P7.50mm_Horizontal"
+		(property "Footprint" "Library:C_Axial_L3.8mm_D2.6mm_P7.50mm_Horizontal_Disc3DModel"
 			(at 18.7452 50.8 0)
 			(effects
@@
 			)
 		)
-		(property "Footprint" "Potentiometer_THT:Potentiometer_Runtron_RM-065_Vertical"
+		(property "Footprint" "Library:Potentiometer_Runtron_RM-065_Vertical_With3DModel"
 			(at 25.4 110.49 0)
 			(effects
@@
 			)
 		)
-		(property "Footprint" "Potentiometer_THT:Potentiometer_Runtron_RM-065_Vertical"
+		(property "Footprint" "Library:Potentiometer_Runtron_RM-065_Vertical_With3DModel"
 			(at 73.66 66.04 0)
 			(effects
@@
 			)
 		)
-		(property "Footprint" "LED_THT:LED_D5.0mm"
+		(property "Footprint" "Library:LED_D5.0mm_Lowered"
 			(at 102.87 86.36 0)
 			(effects
@@
 			)
 		)
-		(property "Footprint" "LED_THT:LED_D5.0mm"
+		(property "Footprint" "Library:LED_D5.0mm_Lowered"
 			(at 102.87 130.81 0)
 			(effects
@@
 			)
 		)
-		(property "Footprint" "Capacitor_THT:C_Axial_L3.8mm_D2.6mm_P7.50mm_Horizontal"
+		(property "Footprint" "Library:C_Axial_L3.8mm_D2.6mm_P7.50mm_Horizontal_Disc3DModel"
 			(at 261.3152 36.83 0)
 			(effects
@@
 			)
 		)
-		(property "Footprint" "Potentiometer_THT:Potentiometer_Runtron_RM-065_Vertical"
+		(property "Footprint" "Library:Potentiometer_Runtron_RM-065_Vertical_With3DModel"
 			(at 73.66 110.49 0)
 			(effects
@@
 			)
 		)
-		(property "Footprint" "Potentiometer_THT:Potentiometer_Runtron_RM-065_Vertical"
+		(property "Footprint" "Library:Potentiometer_Runtron_RM-065_Vertical_With3DModel"
 			(at 73.66 21.59 0)
 			(effects
@@
 			)
 		)
-		(property "Footprint" "Capacitor_THT:C_Axial_L3.8mm_D2.6mm_P7.50mm_Horizontal"
+		(property "Footprint" "Library:C_Axial_L3.8mm_D2.6mm_P7.50mm_Horizontal_Disc3DModel"
 			(at 186.69 40.9448 0)
 			(effects
@@
 			)
 		)
-		(property "Footprint" "Capacitor_THT:C_Axial_L3.8mm_D2.6mm_P7.50mm_Horizontal"
+		(property "Footprint" "Library:C_Axial_L3.8mm_D2.6mm_P7.50mm_Horizontal_Disc3DModel"
 			(at 67.0052 50.8 0)
 			(effects
@@
 			)
 		)
-		(property "Footprint" "Capacitor_THT:C_Axial_L3.8mm_D2.6mm_P7.50mm_Horizontal"
+		(property "Footprint" "Library:C_Axial_L3.8mm_D2.6mm_P7.50mm_Horizontal_Disc3DModel"
 			(at 67.0052 139.7 0)
 			(effects
@@
 			)
 		)
-		(property "Footprint" "LED_THT:LED_D5.0mm"
+		(property "Footprint" "Library:LED_D5.0mm_Lowered"
 			(at 54.61 41.91 0)
 			(effects
@@
 			)
 		)
-		(property "Footprint" "Capacitor_THT:C_Axial_L3.8mm_D2.6mm_P7.50mm_Horizontal"
+		(property "Footprint" "Library:C_Axial_L3.8mm_D2.6mm_P7.50mm_Horizontal_Disc3DModel"
 			(at 67.0052 95.25 0)
 			(effects
@@
 			)
 		)
-		(property "Footprint" "Capacitor_THT:C_Axial_L3.8mm_D2.6mm_P7.50mm_Horizontal"
+		(property "Footprint" "Library:C_Axial_L3.8mm_D2.6mm_P7.50mm_Horizontal_Disc3DModel"
 			(at 18.7452 95.25 0)
 			(effects
@@
 			)
 		)
-		(property "Footprint" "LED_THT:LED_D5.0mm"
+		(property "Footprint" "Library:LED_D5.0mm_Lowered"
 			(at 54.61 86.36 0)
 			(effects
@@
 			)
 		)
-		(property "Footprint" "LED_THT:LED_D5.0mm"
+		(property "Footprint" "Library:LED_D5.0mm_Lowered"
 			(at 54.61 130.81 0)
 			(effects
@@
 			)
 		)
-		(property "Footprint" "LED_THT:LED_D5.0mm"
+		(property "Footprint" "Library:LED_D5.0mm_Lowered"
 			(at 102.87 41.91 0)
 			(effects
@@
 			)
 		)
-		(property "Footprint" "Capacitor_THT:C_Axial_L3.8mm_D2.6mm_P7.50mm_Horizontal"
+		(property "Footprint" "Library:C_Axial_L3.8mm_D2.6mm_P7.50mm_Horizontal_Disc3DModel"
 			(at 18.7452 139.7 0)
 			(effects
@@
 			)
 		)
-		(property "Footprint" "Capacitor_THT:C_Axial_L3.8mm_D2.6mm_P7.50mm_Horizontal"
+		(property "Footprint" "Library:C_Axial_L3.8mm_D2.6mm_P7.50mm_Horizontal_Disc3DModel"
 			(at 172.4152 41.91 0)
 			(effects
@@
 			)
 		)
-		(property "Footprint" "Potentiometer_THT:Potentiometer_Runtron_RM-065_Vertical"
+		(property "Footprint" "Library:Potentiometer_Runtron_RM-065_Vertical_With3DModel"
 			(at 25.4 21.59 0)
 			(effects
